Commit message: Started trying to add CoG plotting but not yet working

File: ur5_model/meshes/ur5.urdf.xacro (robot description, xacro)
@@ -70,4 +70,10 @@
 <!-- ADDED BY ERIC -->
   <xacro:ur5_robot prefix="ur5/" joint_limited="false"/>
+<!--   <joint name="shoulder_link_CoG_joint" type="fixed">
+    <origin xyz="0 0 0" rpy="0 0 0" />
+    <parent link="ur5/shoulder_link" />
+    <child link="shoulder_link_CoG" />
+  </joint>
+  <link name="shoulder_link_CoG"/> -->
   <xacro:macro name="ur5_robot" params="prefix joint_limited">
     <link name="${prefix}base_link" >
